File: schem/schem.kicad_sch (KiCad schematic)
At the start: 6 parts, among them SW1 SW_SPST, U1 ProMicro, U2 CD74HC4067M, U3 ADS7885, U4 CD74HC4067M, U5 OH49E-S

Commit message: Caps/Num/Scr lock status LEDs
Parts:
- added SW2: SW_DIP_x01, symbol Switch:SW_DIP_x01
Connections:
- net +5V: now also U2.16 (I15), U2.17 (I14), U2.18 (I13), U2.19 (I12), U2.2 (I7), U2.20 (I11), U2.21 (I10), U2.22 (I9), U2.23 (I8), U4.16 (I15), U4.17 (I14), U4.18 (I13)
- net GND: now also SW2.2; no longer U2.16 (I15), U2.17 (I14), U2.18 (I13), U2.19 (I12), U2.2 (I7), U2.20 (I11), U2.21 (I10), U2.22 (I9), U2.23 (I8), U4.16 (I15), U4.17 (I14), U4.18 (I13)
- net RT_ENABLE: now also SW2.1
Other:
- moved on the sheet: SW1
